File: control.brd (EAGLE design)
At the start: 186 x 186 mm, 9 parts

Commit message: Work on the control
Parts:
- added C1, C10, C11, C12, C13, C14, C17, C18, C19, C2, C20, C21, C22, C23, C24, C25, C26, C27, C28, C29, C3, C30, C31, C32, C33, C34, C35, C36, C37, C38, C39, C4, C40, C41, C42, C5, C6, C7, C8, C9: 100nF 16V, CAPACITORS:0603
- added C15, C16: 2.2uF 25V, CAPACITORS:0603
- added CN2: MINI B USB, CONNECTORs:MUSB-05-S-B-SM-A
- added FB2: 600R, INDUCTORS:0603
- added R1, R2: 10k, r_0603:0603
- added R10, R11, R12, R13, R14, R15, R16, R17, R18, R3, R4, R5, R6, R7, R8, R9: 1.0k, r_0603:0603
- added SW1, SW10, SW11, SW12, SW13, SW14, SW15, SW16, SW2, SW3, SW4, SW5, SW6, SW7, SW8, SW9: TACT, ELECTROMECH:TL1100DF160Q
- added U1: STM32H743ZI, ICs:QFP144
- added U2: AS4C8M16SA, ICs:TSOPII_54L_100MIL
- added U4: USBLC6-2SC6, ICs:SOT23-6
- added U5: FT230X, ICs:SSOP16-4MM
Connections:
- new net 3V3: C1.2, C10.2, C11.2, C12.2, C13.2, C14.2, C17.2, C18.2, C19.2, C2.2, C20.2, C21.2, C22.2, C23.2, C24.2, C3.2, C4.2, C5.2, C6.2, C7.2, C8.2, C9.2, R1.2, SW1.1, SW1.2, SW10.1, SW10.2, SW11.1, SW11.2, SW12.1, SW12.2, SW13.1, SW13.2, SW14.1, SW14.2, SW15.1, SW15.2, SW16.1, SW16.2, SW2.1, SW2.2, SW3.1, SW3.2, SW4.1, SW4.2, SW5.1, SW5.2, SW6.1, SW6.2, SW7.1, SW7.2, SW8.1, SW8.2, SW9.1, SW9.2, U1.108, U1.121, U1.131, U1.143, U1.144, U1.17, U1.30, U1.32, U1.33, U1.39, U1.52, U1.6, U1.62, U1.72, U1.84, U1.95, U2.1, U2.14, U2.27, U2.3, U2.43, U2.49, U2.9
- new net FT_3V3_BUS: C26.2, U5.10, U5.11, U5.3
- new net FT_UART_BUS_RX: U5.4
- new net FT_UART_BUS_TX: U5.1
- new net GND: C1.1, C10.1, C11.1, C12.1, C13.1, C14.1, C15.2, C16.2, C17.1, C18.1, C19.1, C2.1, C20.1, C21.1, C22.1, C23.1, C24.1, C25.1, C26.1, C27.1, C28.1, C29.1, C3.1, C30.1, C31.1, C32.1, C33.1, C34.1, C35.1, C36.1, C37.1, C38.1, C39.1, C4.1, C40.1, C41.1, C42.1, C5.1, C6.1, C7.1, C8.1, C9.1, CN2.GND, CN2.SHIELD1, CN2.SHIELD2, CN2.SHIELD3, CN2.SHIELD4, R2.1, U1.107, U1.120, U1.130, U1.16, U1.31, U1.38, U1.51, U1.61, U1.83, U1.94, U2.12, U2.28, U2.41, U2.46, U2.52, U2.54, U2.6, U4.2, U5.13, U5.5, U5.6
- new net N$1: C16.1, U1.71
- new net N$10: U2.13
- new net N$11: U2.42
- new net N$12: U2.44
- new net N$13: U2.45
- new net N$14: U2.47
- new net N$15: U2.48
- new net N$16: U2.50
- new net N$17: U2.51
- new net N$18: U2.53
- new net N$19: U2.38
- new net N$2: C15.1, U1.106
- new net N$20: U2.37
- new net N$21: U2.19
- new net N$22: U2.18
- new net N$23: U2.17
- new net N$24: U2.16
- new net N$25: U2.23
- new net N$26: U2.24
- new net N$27: U2.25
- new net N$28: U2.26
- new net N$29: U2.29
- new net N$3: U2.2
- new net N$30: U2.30
- new net N$31: U2.31
- new net N$32: U2.32
- new net N$33: U2.33
- new net N$34: U2.34
- new net N$35: U2.22
- new net N$36: U2.35
- new net N$37: U2.20
- new net N$38: U2.21
- new net N$39: U2.39
- new net N$4: U2.4
- new net N$40: U2.15
- new net N$41: CN2.D-, U4.4
- new net N$42: CN2.D+, U4.6
- new net N$43: U4.3, U5.9
- new net N$44: U4.1, U5.8
- new net N$45: CN2.VCC, FB2.1
- new net N$46: C25.2, FB2.2, U4.5, U5.12
- new net N$47: C27.2, R3.1
- new net N$48: R3.2, SW1.3, SW1.4
- new net N$49: C28.2, R4.1
- new net N$5: U2.5
- new net N$50: R4.2, SW2.3, SW2.4
- new net N$51: C29.2, R5.1
- new net N$52: R5.2, SW3.3, SW3.4
- new net N$53: C30.2, R6.1
- new net N$54: R6.2, SW4.3, SW4.4
- new net N$55: C31.2, R7.1
- new net N$56: R7.2, SW5.3, SW5.4
- new net N$57: C32.2, R8.1
- new net N$58: R8.2, SW6.3, SW6.4
- new net N$59: C33.2, R9.1
- new net N$6: U2.7
- new net N$60: R9.2, SW7.3, SW7.4
- new net N$61: C34.2, R10.1
- new net N$62: R10.2, SW8.3, SW8.4
- new net N$63: C35.2, R11.1
- new net N$64: R11.2, SW9.3, SW9.4
- new net N$65: C36.2, R12.1
- new net N$66: R12.2, SW10.3, SW10.4
- new net N$67: C37.2, R13.1
- new net N$68: R13.2, SW11.3, SW11.4
- new net N$69: C38.2, R14.1
- new net N$7: U2.8
- new net N$70: R14.2, SW12.3, SW12.4
- new net N$71: C39.2, R15.1
- new net N$72: R15.2, SW13.3, SW13.4
- new net N$73: C40.2, R16.1
- new net N$74: R16.2, SW14.3, SW14.4
- new net N$75: C41.2, R17.1
- new net N$76: R17.2, SW15.3, SW15.4
- new net N$77: C42.2, R18.1
- new net N$78: R18.2, SW16.3, SW16.4
- new net N$8: U2.10
- new net N$9: U2.11
- new net STM_BOOT0: R2.2, U1.138
- new net STM_NRST: R1.1, U1.25

Commit message: Progress on PCBs
Parts:
- removed C14, C17: 100nF 16V, CAPACITORS:0603
- added C43: 100nF 16V, CAPACITORS:0603
- added C44: 2.2uF 25V, CAPACITORS:0603
- added C45: 4.7uF 6.3V, CAPACITORS:0603
- added C46: 1uF 25V, CAPACITORS:0603
- added CN1: 40PIN FPC, CONNECTORs:XF2M40151A
- added D1: 3A 0.77V, DIODES:SOD128
- added L1: 4.7uH, INDUCTORS:SRN6045
- added R19: 2R0, RESISTORS:1206
- added R20: 10k, r_0603:0603
- added U3: TPS61169DCKR, ICs:SOT23-5
- added U6: DCDC 3V3, ICs:PDQE10
- moved CN2 155.8 mm to (86.0, 79.0), flipped to the bottom
- moved C25 148.1 mm to (73.2, 80.2), flipped to the bottom
- moved U5 144.1 mm to (71.2, 85.5), flipped to the bottom
- moved C26 140.6 mm to (69.5, 80.2), flipped to the bottom
- moved FB2 133.2 mm to (65.8, 80.2), flipped to the bottom
- moved U4 132.7 mm to (65.5, 86.2), flipped to the bottom
- moved C1 61.7 mm to (32.9, 51.2), flipped to the bottom, turned to 0 degrees
- moved C2 58.1 mm to (32.9, 45.8), flipped to the bottom, turned to 0 degrees
- moved C3 55.3 mm to (32.9, 38.2), flipped to the bottom, turned to 0 degrees
- moved C4 48.2 mm to (27.8, 32.1), flipped to the bottom
- moved C20 42.2 mm to (63.5, 34.6), flipped to the bottom
- moved R1 42.2 mm to (37.8, 15.6), flipped to the bottom, turned to 180 degrees
- moved C32 41.5 mm to (-10.5, -25.5), flipped to the bottom, turned to 270 degrees
- moved C35 39.6 mm to (39.0, -65.0), flipped to the bottom, turned to 270 degrees
- moved C5 38.9 mm to (21.2, 32.1), flipped to the bottom
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Connections:
- removed net FT_UART_BUS_RX: U5.4
- removed net FT_UART_BUS_TX: U5.1
- removed net N$10: U2.13
- removed net N$11: U2.42
- removed net N$12: U2.44
- removed net N$13: U2.45
- removed net N$14: U2.47
- removed net N$15: U2.48
- removed net N$16: U2.50
- removed net N$17: U2.51
- removed net N$18: U2.53
- removed net N$19: U2.38
- removed net N$20: U2.37
- removed net N$21: U2.19
- removed net N$22: U2.18
- removed net N$23: U2.17
- removed net N$24: U2.16
- removed net N$25: U2.23
- removed net N$26: U2.24
- removed net N$27: U2.25
- removed net N$28: U2.26
- removed net N$29: U2.29
- removed net N$3: U2.2
- removed net N$30: U2.30
- removed net N$31: U2.31
- removed net N$32: U2.32
- removed net N$33: U2.33
- removed net N$34: U2.34
- removed net N$35: U2.22
- removed net N$36: U2.35
- removed net N$37: U2.20
- removed net N$38: U2.21
- removed net N$39: U2.39
- removed net N$4: U2.4
- removed net N$40: U2.15
- removed net N$5: U2.5
- removed net N$6: U2.7
- removed net N$7: U2.8
- removed net N$8: U2.10
- removed net N$9: U2.11
- new net ADC_SPI_!CS: U1.125
- new net ADC_SPI_MISO: U1.124
- new net ADC_SPI_MOSI: U1.43
- new net ADC_SPI_SCLK: U1.41
- new net DAC_I2C_SCL: U1.136
- new net DAC_I2C_SDA: U1.137
- new net DISP_!DE: CN1.34, U1.22
- new net DISP_B0: CN1.21, U1.3
- new net DISP_B1: CN1.22, U1.127
- new net DISP_B2: CN1.23, U1.122
- new net DISP_B3: CN1.24, U1.100
- new net DISP_B4: CN1.25, U1.102
- new net DISP_B5: CN1.26, U1.37
- new net DISP_B6: CN1.27, U1.139
- new net DISP_B7: CN1.28, U1.140
- new net DISP_CLK: CN1.30, U1.92
- new net DISP_DE: U1.18
- new net DISP_G0: CN1.13, U1.4
- new net DISP_G1: CN1.14, U1.5
- new net DISP_G2: CN1.15, U1.42
- new net DISP_G3: CN1.16, U1.117, U1.99
- new net DISP_G4: CN1.17, U1.69
- new net DISP_G5: CN1.18, U1.70
- new net DISP_G6: CN1.19, U1.97
- new net DISP_G7: CN1.20
- new net DISP_HSD: CN1.32, U1.44, U1.96
- new net DISP_LED+: C46.2, CN1.2, D1.K
- new net DISP_LED-: CN1.1, R19.2, U3.3
- new net DISP_PWM: R20.2, U3.4
- new net DISP_R0: CN1.5, U1.128
- new net DISP_R1: CN1.6, U1.36
- new net DISP_R2: CN1.7, U1.35
- new net DISP_R3: CN1.8, U1.46
- new net DISP_R4: CN1.9, U1.103
- new net DISP_R5: CN1.10, U1.101
- new net DISP_R6: CN1.11, U1.47
- new net DISP_R7: CN1.12, U1.91
- new net DISP_STBY: CN1.31
- new net DISP_VSD: CN1.33, U1.40
- new net FT_UART_RX: U1.75, U5.4
- new net FT_UART_TX: U1.76, U5.1
- new net JTAG_TCK: U1.109
- new net JTAG_TDI: U1.110
- new net JTAG_TMS: U1.105
- new net JTAG_TRACE: U1.133
- new net JTAG_TRACECLK: U1.1
- new net JTAG_TRACED0: U1.2
- new net N$101: U1.48
- new net N$103: U1.134
- new net N$104: U1.135
- new net N$111: U1.73
- new net N$112: U1.74
- new net N$120: U1.45
- new net N$123: U1.98
- new net N$125: U1.111
- new net N$126: U1.112
- new net N$127: U1.113
- new net N$128: U1.7
- new net N$129: U1.8
- new net N$130: U1.9
- new net N$133: U1.116
- new net N$135: U1.118
- new net N$136: U1.119
- new net N$138: U1.123
- new net N$142: U1.80
- new net N$143: U1.81
- new net N$144: U1.82
- new net N$161: U1.142
- new net N$162: U1.141
- new net N$169: U1.21
- new net N$170: U1.20
- new net N$171: U1.19
- new net N$180: U1.129
- new net N$183: U1.126
- new net N$191: U1.88
- new net N$192: U1.87
- new net N$83: U1.34
- new net N$84: U1.27
- new net N$86: D1.A, L1.2, U3.1
- new net N$95: U1.104
- new net SDRAM_!CAS: U1.132, U2.17
- new net SDRAM_!CS: U1.28, U2.19
- new net SDRAM_!RAS: U1.49, U2.18
- new net SDRAM_!WE: U1.26, U2.16
- new net SDRAM_A0: U1.10, U2.23
- new net SDRAM_A1: U1.11, U2.24
- new net SDRAM_A10: U1.56, U2.22
- new net SDRAM_A11: U1.57, U2.35
- new net SDRAM_A2: U1.12, U2.25
- new net SDRAM_A3: U1.13, U2.26
- new net SDRAM_A4: U1.14, U2.29
- new net SDRAM_A5: U1.15, U2.30
- new net SDRAM_A6: U1.50, U2.31
- new net SDRAM_A7: U1.53, U2.32
- new net SDRAM_A8: U1.54, U2.33
- new net SDRAM_A9: U1.55, U2.34
- new net SDRAM_BA0: U1.89, U2.20
- new net SDRAM_BA1: U1.90, U2.21
- new net SDRAM_CKE: U1.29, U2.37
- new net SDRAM_CLK: U1.93, U2.38
- new net SDRAM_D0: U1.85, U2.2
- new net SDRAM_D1: U1.86, U2.4
- new net SDRAM_D10: U1.66, U2.45
- new net SDRAM_D11: U1.67, U2.47
- new net SDRAM_D12: U1.68, U2.48
- new net SDRAM_D13: U1.77, U2.50
- new net SDRAM_D14: U1.78, U2.51
- new net SDRAM_D15: U1.79, U2.53
- new net SDRAM_D2: U1.114, U2.5
- new net SDRAM_D3: U1.115, U2.7
- new net SDRAM_D4: U1.58, U2.8
- new net SDRAM_D5: U1.59, U2.10
- new net SDRAM_D6: U1.60, U2.11
- new net SDRAM_D7: U1.63, U2.13
- new net SDRAM_D8: U1.64, U2.42
- new net SDRAM_D9: U1.65, U2.44
- net 3V3: now also C43.2, C44.2, C45.2, CN1.4, L1.1, U2.15, U2.39, U3.5; no longer C14.2, C17.2
- net GND: now also C43.1, C44.1, C45.1, C46.1, CN1.29, CN1.3, CN1.36, R19.1, R20.1, U3.2; no longer C14.1, C17.1
Routing:
- net 3V3: track 0.00 -> 61.4 mm, vias 0 -> 24
- net GND: track 0.00 -> 53.8 mm, vias 0 -> 52
- net N$82: track 0.00 -> 10.0 mm
- net N$81: track 0.00 -> 10.0 mm
- net N$80: track 0.00 -> 10.0 mm
- net N$79: track 0.00 -> 10.0 mm
- net DISP_LED+: track 0.00 -> 2.60 mm
- net N$1: track 0.00 -> 1.81 mm
- net N$2: track 0.00 -> 1.60 mm
- net DISP_LED-: track 0.00 -> 1.12 mm
- added copper zone on layer 2, net 3V3
- added copper zone on layer 3, net GND
Other:
- outline, holes or cut-outs redrawn

Commit message: Progress
Parts:
- added CN3: 0530471210, CONNECTORs:MOLEX_530471210
- moved CN2 172.0 mm to (-86.0, 81.0)
- moved U6 153.5 mm to (75.2, 71.5)
- moved C25 141.0 mm to (-67.8, 81.2)
- moved C26 141.0 mm to (-71.5, 81.2)
- moved FB2 141.0 mm to (-75.2, 81.2)
- moved U4 141.0 mm to (-75.5, 87.2)
- moved U5 141.0 mm to (-69.8, 86.5)
Connections:
- new net 3V3D: CN3.3, CN3.4
- new net ADC_!DRDY: CN3.7
- new net DGND: CN3.10, CN3.11, CN3.12
- net ADC_SPI_!CS: now also CN3.8
- net ADC_SPI_MISO: now also CN3.6
- net ADC_SPI_MOSI: now also CN3.5
- net ADC_SPI_SCLK: now also CN3.9
- net DAC_I2C_SCL: now also CN3.1
- net DAC_I2C_SDA: now also CN3.2
Routing:
- net SDRAM_BA0: track 0.00 -> 99.4 mm, vias 0 -> 4
- net SDRAM_BA1: track 0.00 -> 97.2 mm, vias 0 -> 4
- net SDRAM_D6: track 0.00 -> 83.0 mm, vias 0 -> 4
- net SDRAM_D4: track 0.00 -> 82.5 mm, vias 0 -> 4
- net SDRAM_D5: track 0.00 -> 82.3 mm, vias 0 -> 4
- net SDRAM_D7: track 0.00 -> 81.8 mm, vias 0 -> 4
- net SDRAM_D12: track 0.00 -> 77.7 mm, vias 0 -> 4
- net SDRAM_D11: track 0.00 -> 72.3 mm, vias 0 -> 4
- net SDRAM_!RAS: track 0.00 -> 67.9 mm, vias 0 -> 4
- net SDRAM_D9: track 0.00 -> 67.2 mm, vias 0 -> 4
- net SDRAM_!CAS: track 0.00 -> 67.2 mm, vias 0 -> 4
- net SDRAM_A10: track 0.00 -> 65.2 mm, vias 0 -> 4
- net SDRAM_!WE: track 0.00 -> 63.5 mm, vias 0 -> 4
- net SDRAM_D10: track 0.00 -> 57.6 mm, vias 0 -> 4
- net SDRAM_D8: track 0.00 -> 55.3 mm, vias 0 -> 4
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Other:
- outline, holes or cut-outs redrawn

Commit message: Progress
Parts:
- added TP1, TP2: TEST_POINT_SQUARE, MISC:OSPREY_HSS_PAD
- moved CN3 149.0 mm to (75.0, 5.00), flipped to the bottom, turned to 180 degrees
- moved R1 63.7 mm to (19.8, 76.8)
- moved U6 36.8 mm to (80.0, 35.0)
- moved R2 22.2 mm to (25.8, 57.9), turned to 270 degrees
- moved D1 12.6 mm to (-41.4, 35.8), turned to 270 degrees
- moved C46 12.5 mm to (-41.4, 31.1), turned to 90 degrees
- moved L1 11.2 mm to (-49.6, 41.9), turned to 180 degrees
- moved C45 10.6 mm to (-53.8, 40.0), turned to 270 degrees
- moved C26 9.50 mm to (-62.6, 84.6)
- moved U3 7.77 mm to (-51.0, 37.1), turned to 90 degrees
- moved FB2 6.79 mm to (-76.8, 87.9), turned to 180 degrees
- moved C25 5.55 mm to (-62.6, 83.4)
- moved R20 5.14 mm to (-51.8, 35.0)
- moved R19 4.85 mm to (-44.4, 34.8), turned to 270 degrees
- moved U5 4.16 mm to (-67.5, 83.0), turned to 180 degrees
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Connections:
- removed net N$83: U1.34
- new net N$3: U1.44
- new net N$4: TP1.1, U6.2
- new net N$5: TP2.1, U6.1
- net 3V3: now also U6.3
- net DISP_G3: no longer U1.117
- net DISP_G7: now also U1.117
- net DISP_HSD: no longer U1.44
- net DISP_PWM: now also U1.34
- net GND: now also U6.5
Routing:
- net DAC_I2C_SCL: track 0.00 -> 138.5 mm, vias 0 -> 3
- net ADC_SPI_MISO: track 0.00 -> 136.2 mm, vias 0 -> 3
- net DAC_I2C_SDA: track 0.00 -> 135.3 mm, vias 0 -> 3
- net ADC_SPI_!CS: track 0.00 -> 132.2 mm, vias 0 -> 3
- net DISP_PWM: track 0.00 -> 123.4 mm, vias 0 -> 4
- net FT_UART_RX: track 0.00 -> 117.5 mm, vias 0 -> 2
- net FT_UART_TX: track 0.00 -> 117.0 mm, vias 0 -> 2
- net DISP_!DE: track 0.00 -> 114.6 mm, vias 0 -> 4
- net DISP_G0: track 0.00 -> 112.1 mm, vias 0 -> 4
- net DISP_G1: track 0.00 -> 110.2 mm, vias 0 -> 4
- net DISP_B0: track 0.00 -> 109.6 mm, vias 0 -> 4
- net SDRAM_D1: track 0.00 -> 107.6 mm, vias 0 -> 4
- net DISP_R2: track 0.00 -> 106.9 mm, vias 0 -> 4
- net SDRAM_D0: track 0.00 -> 106.6 mm, vias 0 -> 4
- net SDRAM_D13: track 0.00 -> 105.9 mm, vias 0 -> 4
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
Commit message: Control nearly done
Parts:
- removed TP1, TP2: TEST_POINT_SQUARE, MISC:OSPREY_HSS_PAD
- added CN4: 2X10 HEADER, CONNECTORs:2X10PIN_HEADER
- added R21: 10R, r_0603:0603
- CN3: value 0530471210 -> 2X10 HEADER; device CONNECTORs:MOLEX_530471210 -> CONNECTORs:2X10PIN_HEADER
- moved CN3 156.6 mm to (-75.0, 50.0), flipped to the top, turned to 0 degrees
- moved C35 49.3 mm to (21.9, -18.8), turned to 180 degrees
- moved R14 49.2 mm to (46.9, -17.5), turned to 0 degrees
- moved R5 46.0 mm to (-28.1, -17.5), turned to 0 degrees
- moved C29 45.2 mm to (-28.1, -18.8)
- moved C31 40.8 mm to (-28.2, -68.8)
- moved R8 40.3 mm to (-3.25, -17.5), turned to 0 degrees
- moved C40 39.3 mm to (46.9, -68.8), turned to 180 degrees
- moved R7 39.0 mm to (-28.2, -67.5), turned to 0 degrees
- moved R1 37.4 mm to (32.9, 41.8)
- moved C34 36.5 mm to (-3.25, -68.8), turned to 180 degrees
- moved C37 36.0 mm to (21.9, -68.8), turned to 180 degrees
- moved C38 35.9 mm to (46.9, -18.8), turned to 180 degrees
- moved R15 35.2 mm to (46.9, -42.5), turned to 0 degrees
- moved R16 31.2 mm to (46.9, -67.5), turned to 0 degrees
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Connections:
- net JTAG_TRACECLK renamed N$5
- net JTAG_TRACED0 renamed N$6
- removed net 3V3D: CN3.3, CN3.4
- removed net DGND: CN3.10, CN3.11, CN3.12
- removed net DISP_!DE: CN1.34, U1.22
- removed net DISP_STBY: CN1.31
- removed net JTAG_TRACE: U1.133
- removed net N$101: U1.48
- removed net N$103: U1.134
- removed net N$111: U1.73
- removed net N$112: U1.74
- removed net N$120: U1.45
- removed net N$123: U1.98
- removed net N$128: U1.7
- removed net N$129: U1.8
- removed net N$130: U1.9
- removed net N$142: U1.80
- removed net N$143: U1.81
- removed net N$144: U1.82
- removed net N$169: U1.21
- removed net N$170: U1.20
- removed net N$171: U1.19
- removed net N$191: U1.88
- removed net N$192: U1.87
- removed net N$3: U1.44
- removed net N$47: C27.2, R3.1
- removed net N$49: C28.2, R4.1
- removed net N$5 (its old number): TP2.1, U6.1
- removed net N$51: C29.2, R5.1
- removed net N$53: C30.2, R6.1
- removed net N$55: C31.2, R7.1
- removed net N$57: C32.2, R8.1
- removed net N$59: C33.2, R9.1
- removed net N$61: C34.2, R10.1
- removed net N$63: C35.2, R11.1
- removed net N$65: C36.2, R12.1
- removed net N$67: C37.2, R13.1
- removed net N$69: C38.2, R14.1
- removed net N$71: C39.2, R15.1
- removed net N$73: C40.2, R16.1
- removed net N$75: C41.2, R17.1
- removed net N$77: C42.2, R18.1
- new net BTN_0: C40.2, R16.1, U1.9
- new net BTN_1: C31.2, R7.1, U1.80
- new net BTN_2: C34.2, R10.1, R21.2, U1.21
- new net BTN_3: C37.2, R13.1, U1.19
- new net BTN_4: C30.2, R6.1, U1.81
- new net BTN_5: C33.2, R9.1, U1.73
- new net BTN_6: C36.2, R12.1, U1.44
- new net BTN_7: C29.2, R5.1, U1.82
- new net BTN_8: C32.2, R8.1, U1.74
- new net BTN_9: C35.2, R11.1, U1.20
- new net BTN_AMPS: C41.2, R17.1, U1.7
- new net BTN_CANCEL: C38.2, R14.1, U1.8
- new net BTN_DP: C39.2, R15.1, U1.45
- new net BTN_ON0FF: C27.2, R3.1, U1.88
- new net BTN_OUT_CONT: C28.2, R4.1, U1.87
- new net BTN_VOLTS: C42.2, R18.1, U1.48
- new net DISP_EN: CN1.31, U1.98
- new net JTAG_TDO: CN3.7, U1.133
- new net JTAG_TRST: CN3.2, U1.134
- new net PGND: CN4.10, CN4.11, CN4.12, CN4.9, U6.1
- new net VIN: CN4.13, CN4.14, CN4.7, CN4.8, U6.2
- net 3V3: now also CN3.1, CN4.19, CN4.2
- net ADC_!DRDY: now also CN4.5; no longer CN3.7
- net ADC_SPI_!CS: now also CN4.15; no longer CN3.8
- net ADC_SPI_MISO: now also CN4.4; no longer CN3.6
- net ADC_SPI_MOSI: now also CN4.3; no longer CN3.5
- net ADC_SPI_SCLK: now also CN4.6; no longer CN3.9
- net DAC_I2C_SCL: now also CN4.17; no longer CN3.1
- net DAC_I2C_SDA: now also CN4.18; no longer CN3.2
- net DISP_DE: now also CN1.34, U1.22; no longer U1.18
- net GND: now also CN3.11, CN3.12, CN3.13, CN3.14, CN3.15, CN3.16, CN3.17, CN3.18, CN3.19, CN3.6, CN4.1, CN4.16, CN4.20
- net JTAG_TCK: now also CN3.5
- net JTAG_TDI: now also CN3.3
- net JTAG_TMS: now also CN3.4
- net N$4: now also U1.18; no longer TP1.1, U6.2
- net STM_BOOT0: now also R21.1
- net STM_NRST: now also CN3.8
Routing:
- net BTN_OUT_CONT: track 0.00 -> 203.8 mm, vias 0 -> 4
- net BTN_2: track 0.00 -> 188.5 mm, vias 0 -> 6
- net BTN_1: track 0.00 -> 186.7 mm, vias 0 -> 4
- net BTN_ON0FF: track 0.00 -> 180.6 mm, vias 0 -> 4
- net STM_NRST: track 0.00 -> 165.8 mm, vias 0 -> 6
- net BTN_4: track 0.00 -> 162.5 mm, vias 0 -> 4
- net BTN_7: track 0.00 -> 138.2 mm, vias 0 -> 4
- net BTN_5: track 0.00 -> 133.6 mm, vias 0 -> 4
- net JTAG_TRST: track 0.00 -> 131.0 mm, vias 0 -> 4
- net BTN_0: track 0.00 -> 128.5 mm, vias 0 -> 2
- net BTN_3: track 0.00 -> 123.2 mm, vias 0 -> 2
- net BTN_VOLTS: track 0.00 -> 122.2 mm, vias 0 -> 4
- net JTAG_TDO: track 0.00 -> 120.6 mm, vias 0 -> 4
- net DISP_DE: track 0.00 -> 114.6 mm, vias 0 -> 4
- net DISP_!DE: track 114.6 -> 0.00 mm, vias 4 -> 0
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