File: control.sch (EAGLE design)
At the start: 9 parts

Commit message: Work on the control
Parts:
- added C1, C10, C11, C12, C13, C14, C17, C18, C19, C2, C20, C21, C22, C23, C24, C25, C26, C27, C28, C29, C3, C30, C31, C32, C33, C34, C35, C36, C37, C38, C39, C4, C40, C41, C42, C5, C6, C7, C8, C9: 100nF 16V, CAPACITORS:CL10B104KO8WPNC
- added C15, C16: 2.2uF 25V, CAPACITORS:GRM188R61E225KA12D
- added CN2: MINI B USB, CONNECTORs:MUSB-05-S-B-SM-A
- added FB2: 600R, INDUCTORS:742792651
- added R1, R2: 10k, r_0603:ERJ3EKF1002V
- added R10, R11, R12, R13, R14, R15, R16, R17, R18, R3, R4, R5, R6, R7, R8, R9: 1.0k, r_0603:ERJ3EKF1001V
- added SW1, SW10, SW11, SW12, SW13, SW14, SW15, SW16, SW2, SW3, SW4, SW5, SW6, SW7, SW8, SW9: TACT, ELECTROMECH:TL1100DF160Q
- added U1: STM32H743ZI, ICs:STM32H743ZI
- added U2: AS4C8M16SA, ICs:AS4C8M16SA
- added U4: USBLC6-2SC6, ICs:USBLC6-2SC6
- added U5: FT230X, ICs:FT230XS
Connections:
- new net 3V3: C1.2, C10.2, C11.2, C12.2, C13.2, C14.2, C17.2, C18.2, C19.2, C2.2, C20.2, C21.2, C22.2, C23.2, C24.2, C3.2, C4.2, C5.2, C6.2, C7.2, C8.2, C9.2, R1.2, SW1.1, SW10.1, SW11.1, SW12.1, SW13.1, SW14.1, SW15.1, SW16.1, SW2.1, SW3.1, SW4.1, SW5.1, SW6.1, SW7.1, SW8.1, SW9.1, U1.PDR_ON, U1.VBAT, U1.VDD, U1.VDD33_USB, U1.VDDA, U1.VREF+, U2.VDD, U2.VDDQ
- new net FT_3V3_BUS: C26.2, U5.!RESET, U5.3V3OUT, U5.VCCIO
- new net FT_UART_BUS_RX: U5.RXD
- new net FT_UART_BUS_TX: U5.TXD
- new net GND: C1.1, C10.1, C11.1, C12.1, C13.1, C14.1, C15.2, C16.2, C17.1, C18.1, C19.1, C2.1, C20.1, C21.1, C22.1, C23.1, C24.1, C25.1, C26.1, C27.1, C28.1, C29.1, C3.1, C30.1, C31.1, C32.1, C33.1, C34.1, C35.1, C36.1, C37.1, C38.1, C39.1, C4.1, C40.1, C41.1, C42.1, C5.1, C6.1, C7.1, C8.1, C9.1, CN2.GND, R2.1, U1.VSS, U1.VSSA, U2.VSS, U2.VSSQ, U4.GND, U5.!CTS, U5.GND
- new net N$1: C16.1, U1.VCAP1
- new net N$10: U2.D7
- new net N$11: U2.D8
- new net N$12: U2.D9
- new net N$13: U2.D10
- new net N$14: U2.D11
- new net N$15: U2.D12
- new net N$16: U2.D13
- new net N$17: U2.D14
- new net N$18: U2.D15
- new net N$19: U2.CLK
- new net N$2: C15.1, U1.VCAP2
- new net N$20: U2.CKE
- new net N$21: U2.!CS
- new net N$22: U2.!RAS
- new net N$23: U2.!CAS
- new net N$24: U2.!WE
- new net N$25: U2.A0
- new net N$26: U2.A1
- new net N$27: U2.A2
- new net N$28: U2.A3
- new net N$29: U2.A4
- new net N$3: U2.D0
- new net N$30: U2.A5
- new net N$31: U2.A6
- new net N$32: U2.A7
- new net N$33: U2.A8
- new net N$34: U2.A9
- new net N$35: U2.A10
- new net N$36: U2.A11
- new net N$37: U2.BA0
- new net N$38: U2.BA1
- new net N$39: U2.UDM
- new net N$4: U2.D1
- new net N$40: U2.LDM
- new net N$41: CN2.D-, U4.D-OUT
- new net N$42: CN2.D+, U4.D+_OUT
- new net N$43: U4.D-_IN, U5.D-
- new net N$44: U4.D+_IN, U5.D+
- new net N$45: CN2.5V, FB2.1
- new net N$46: C25.2, FB2.2, U4.VBUS, U5.VCC
- new net N$47: C27.2, R3.1
- new net N$48: R3.2, SW1.2
- new net N$49: C28.2, R4.1
- new net N$5: U2.D2
- new net N$50: R4.2, SW2.2
- new net N$51: C29.2, R5.1
- new net N$52: R5.2, SW3.2
- new net N$53: C30.2, R6.1
- new net N$54: R6.2, SW4.2
- new net N$55: C31.2, R7.1
- new net N$56: R7.2, SW5.2
- new net N$57: C32.2, R8.1
- new net N$58: R8.2, SW6.2
- new net N$59: C33.2, R9.1
- new net N$6: U2.D3
- new net N$60: R9.2, SW7.2
- new net N$61: C34.2, R10.1
- new net N$62: R10.2, SW8.2
- new net N$63: C35.2, R11.1
- new net N$64: R11.2, SW9.2
- new net N$65: C36.2, R12.1
- new net N$66: R12.2, SW10.2
- new net N$67: C37.2, R13.1
- new net N$68: R13.2, SW11.2
- new net N$69: C38.2, R14.1
- new net N$7: U2.D4
- new net N$70: R14.2, SW12.2
- new net N$71: C39.2, R15.1
- new net N$72: R15.2, SW13.2
- new net N$73: C40.2, R16.1
- new net N$74: R16.2, SW14.2
- new net N$75: C41.2, R17.1
- new net N$76: R17.2, SW15.2
- new net N$77: C42.2, R18.1
- new net N$78: R18.2, SW16.2
- new net N$8: U2.D5
- new net N$9: U2.D6
- new net STM_BOOT0: R2.2, U1.BOOT0
- new net STM_NRST: R1.1, U1.NRST

Commit message: Progress on PCBs
Parts:
- removed C14, C17: 100nF 16V, CAPACITORS:CL10B104KO8WPNC
- added C43: 100nF 16V, CAPACITORS:CL10B104KO8WPNC
- added C44: 2.2uF 25V, CAPACITORS:GRM188R61E225KA12D
- added C45: 4.7uF 6.3V, CAPACITORS:GRM188R60J475ME19D
- added C46: 1uF 25V, CAPACITORS:CL10A105KA8NNNC
- added CN1: 40PIN FPC, CONNECTORs:XF2M40151A
- added D1: 3A 0.77V, DIODES:PMEG10030ELP
- added L1: 4.7uH, INDUCTORS:SRN6045TA-4R7M
- added R19: 2R0, RESISTORS:CRCW12062R00FNEA
- added R20: 10k, r_0603:ERJ3EKF1002V
- added U3: TPS61169DCKR, ICs:TPS61169DCKR
- added U6: DCDC 3V3, ICs:PDQE15-Q24-S3-D
Connections:
- removed net FT_UART_BUS_RX: U5.RXD
- removed net FT_UART_BUS_TX: U5.TXD
- removed net N$10: U2.D7
- removed net N$11: U2.D8
- removed net N$12: U2.D9
- removed net N$13: U2.D10
- removed net N$14: U2.D11
- removed net N$15: U2.D12
- removed net N$16: U2.D13
- removed net N$17: U2.D14
- removed net N$18: U2.D15
- removed net N$19: U2.CLK
- removed net N$20: U2.CKE
- removed net N$21: U2.!CS
- removed net N$22: U2.!RAS
- removed net N$23: U2.!CAS
- removed net N$24: U2.!WE
- removed net N$25: U2.A0
- removed net N$26: U2.A1
- removed net N$27: U2.A2
- removed net N$28: U2.A3
- removed net N$29: U2.A4
- removed net N$3: U2.D0
- removed net N$30: U2.A5
- removed net N$31: U2.A6
- removed net N$32: U2.A7
- removed net N$33: U2.A8
- removed net N$34: U2.A9
- removed net N$35: U2.A10
- removed net N$36: U2.A11
- removed net N$37: U2.BA0
- removed net N$38: U2.BA1
- removed net N$39: U2.UDM
- removed net N$4: U2.D1
- removed net N$40: U2.LDM
- removed net N$5: U2.D2
- removed net N$6: U2.D3
- removed net N$7: U2.D4
- removed net N$8: U2.D5
- removed net N$9: U2.D6
- new net ADC_SPI_!CS: U1.PG10
- new net ADC_SPI_MISO: U1.PG9
- new net ADC_SPI_MOSI: U1.PA7
- new net ADC_SPI_SCLK: U1.PA5
- new net DAC_I2C_SCL: U1.PB6
- new net DAC_I2C_SDA: U1.PB7
- new net DISP_!DE: CN1.34, U1.PF10
- new net DISP_B0: CN1.21, U1.PE4
- new net DISP_B1: CN1.22, U1.PG12
- new net DISP_B2: CN1.23, U1.PD6
- new net DISP_B3: CN1.24, U1.PA8
- new net DISP_B4: CN1.25, U1.PA10
- new net DISP_B5: CN1.26, U1.PA3
- new net DISP_B6: CN1.27, U1.PB8
- new net DISP_B7: CN1.28, U1.PB9
- new net DISP_CLK: CN1.30, U1.PG7
- new net DISP_DE: U1.PF6
- new net DISP_G0: CN1.13, U1.PE5
- new net DISP_G1: CN1.14, U1.PE6
- new net DISP_G2: CN1.15, U1.PA6
- new net DISP_G3: CN1.16, U1.PC9, U1.PD3
- new net DISP_G4: CN1.17, U1.PB10
- new net DISP_G5: CN1.18, U1.PB11
- new net DISP_G6: CN1.19, U1.PC7
- new net DISP_G7: CN1.20
- new net DISP_HSD: CN1.32, U1.PC4, U1.PC6
- new net DISP_LED+: C46.2, CN1.2, D1.K
- new net DISP_LED-: CN1.1, R19.2, U3.FB
- new net DISP_PWM: R20.2, U3.CTRL
- new net DISP_R0: CN1.5, U1.PG13
- new net DISP_R1: CN1.6, U1.PA2
- new net DISP_R2: CN1.7, U1.PA1
- new net DISP_R3: CN1.8, U1.PB0
- new net DISP_R4: CN1.9, U1.PA11
- new net DISP_R5: CN1.10, U1.PA9
- new net DISP_R6: CN1.11, U1.PB1
- new net DISP_R7: CN1.12, U1.PG6
- new net DISP_STBY: CN1.31
- new net DISP_VSD: CN1.33, U1.PA4
- new net FT_UART_RX: U1.PB14, U5.RXD
- new net FT_UART_TX: U1.PB15, U5.TXD
- new net JTAG_TCK: U1.PA14
- new net JTAG_TDI: U1.PA15
- new net JTAG_TMS: U1.PA13
- new net JTAG_TRACE: U1.PB3
- new net JTAG_TRACECLK: U1.PE2
- new net JTAG_TRACED0: U1.PE3
- new net N$101: U1.PB2
- new net N$103: U1.PB4
- new net N$104: U1.PB5
- new net N$111: U1.PB12
- new net N$112: U1.PB13
- new net N$120: U1.PC5
- new net N$123: U1.PC8
- new net N$125: U1.PC10
- new net N$126: U1.PC11
- new net N$127: U1.PC12
- new net N$128: U1.PC13
- new net N$129: U1.PC14
- new net N$130: U1.PC15
- new net N$133: U1.PD2
- new net N$135: U1.PD4
- new net N$136: U1.PD5
- new net N$138: U1.PD7
- new net N$142: U1.PD11
- new net N$143: U1.PD12
- new net N$144: U1.PD13
- new net N$161: U1.PE1
- new net N$162: U1.PE0
- new net N$169: U1.PF9
- new net N$170: U1.PF8
- new net N$171: U1.PF7
- new net N$180: U1.PG14
- new net N$183: U1.PG11
- new net N$191: U1.PG3
- new net N$192: U1.PG2
- new net N$83: U1.PA0
- new net N$84: U1.PC1
- new net N$86: D1.A, L1.2, U3.SW
- new net N$95: U1.PA12
- new net SDRAM_!CAS: U1.PG15, U2.!CAS
- new net SDRAM_!CS: U1.PC2, U2.!CS
- new net SDRAM_!RAS: U1.PF11, U2.!RAS
- new net SDRAM_!WE: U1.PC0, U2.!WE
- new net SDRAM_A0: U1.PF0, U2.A0
- new net SDRAM_A1: U1.PF1, U2.A1
- new net SDRAM_A10: U1.PG0, U2.A10
- new net SDRAM_A11: U1.PG1, U2.A11
- new net SDRAM_A2: U1.PF2, U2.A2
- new net SDRAM_A3: U1.PF3, U2.A3
- new net SDRAM_A4: U1.PF4, U2.A4
- new net SDRAM_A5: U1.PF5, U2.A5
- new net SDRAM_A6: U1.PF12, U2.A6
- new net SDRAM_A7: U1.PF13, U2.A7
- new net SDRAM_A8: U1.PF14, U2.A8
- new net SDRAM_A9: U1.PF15, U2.A9
- new net SDRAM_BA0: U1.PG4, U2.BA0
- new net SDRAM_BA1: U1.PG5, U2.BA1
- new net SDRAM_CKE: U1.PC3, U2.CKE
- new net SDRAM_CLK: U1.PG8, U2.CLK
- new net SDRAM_D0: U1.PD14, U2.D0
- new net SDRAM_D1: U1.PD15, U2.D1
- new net SDRAM_D10: U1.PE13, U2.D10
- new net SDRAM_D11: U1.PE14, U2.D11
- new net SDRAM_D12: U1.PE15, U2.D12
- new net SDRAM_D13: U1.PD8, U2.D13
- new net SDRAM_D14: U1.PD9, U2.D14
- new net SDRAM_D15: U1.PD10, U2.D15
- new net SDRAM_D2: U1.PD0, U2.D2
- new net SDRAM_D3: U1.PD1, U2.D3
- new net SDRAM_D4: U1.PE7, U2.D4
- new net SDRAM_D5: U1.PE8, U2.D5
- new net SDRAM_D6: U1.PE9, U2.D6
- new net SDRAM_D7: U1.PE10, U2.D7
- new net SDRAM_D8: U1.PE11, U2.D8
- new net SDRAM_D9: U1.PE12, U2.D9
- net 3V3: now also C43.2, C44.2, C45.2, CN1.4, L1.1, U2.LDM, U2.UDM, U3.VIN; no longer C14.2, C17.2
- net GND: now also C43.1, C44.1, C45.1, C46.1, CN1.29, CN1.3, CN1.36, R19.1, R20.1, U3.GND; no longer C14.1, C17.1
Other:
- moved on the sheet: C18, C19, C20, C21, C22, C23, C24, U2

Commit message: Progress
Parts:
- added CN3: 0530471210, CONNECTORs:PICOBLADE_12_TH_V
Connections:
- new net 3V3D: CN3.3, CN3.4
- new net ADC_!DRDY: CN3.7
- new net DGND: CN3.10, CN3.11, CN3.12
- net ADC_SPI_!CS: now also CN3.8
- net ADC_SPI_MISO: now also CN3.6
- net ADC_SPI_MOSI: now also CN3.5
- net ADC_SPI_SCLK: now also CN3.9
- net DAC_I2C_SCL: now also CN3.1
- net DAC_I2C_SDA: now also CN3.2
Changed lines of the file:
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@@
 <part name="GND54" library="NETS" deviceset="GND" device=""/>
 <part name="U$43" library="NETS" deviceset="3V3" device=""/>
+<part name="CN3" library="CONNECTORs" deviceset="PICOBLADE_12_" device="TH_V" value="0530471210"/>
 </parts>
 <sheets>
@@
 <instance part="U$43" gate="G$1" x="-35.56" y="76.2" smashed="yes">
 <attribute name="VALUE" x="-35.56" y="78.74" size="1.778" layer="96" rot="R180" align="center"/>
+</instance>
+<instance part="CN3" gate="G$1" x="231.14" y="325.12" smashed="yes">
+<attribute name="NAME" x="226.06" y="345.44" size="2.286" layer="95"/>
+<attribute name="VALUE" x="226.06" y="342.9" size="2.286" layer="96"/>
 </instance>
 </instances>
@@
 <label x="76.2" y="243.84" size="1.778" layer="95"/>
 </segment>
+<segment>
+<pinref part="CN3" gate="G$1" pin="9"/>
+<wire x1="238.76" y1="317.5" x2="271.78" y2="317.5" width="0.1524" layer="91"/>
+<label x="241.3" y="317.5" size="1.778" layer="95"/>
+</segment>
 </net>
 <net name="ADC_SPI_MOSI" class="0">
@@
 <label x="76.2" y="238.76" size="1.778" layer="95"/>
 </segment>
+<segment>
+<pinref part="CN3" gate="G$1" pin="5"/>
+<wire x1="238.76" y1="327.66" x2="271.78" y2="327.66" width="0.1524" layer="91"/>
+<label x="241.3" y="327.66" size="1.778" layer="95"/>
+</segment>
 </net>
 <net name="N$95" class="0">
@@
 <label x="76.2" y="198.12" size="1.778" layer="95"/>
 </segment>
+<segment>
+<pinref part="CN3" gate="G$1" pin="1"/>
+<wire x1="238.76" y1="337.82" x2="271.78" y2="337.82" width="0.1524" layer="91"/>
+<label x="241.3" y="337.82" size="1.778" layer="95"/>
+</segment>
 </net>
 <net name="DAC_I2C_SDA" class="0">
@@
 <label x="76.2" y="195.58" size="1.778" layer="95"/>
 </segment>
+<segment>
+<pinref part="CN3" gate="G$1" pin="2"/>
+<wire x1="238.76" y1="335.28" x2="271.78" y2="335.28" width="0.1524" layer="91"/>
+<label x="241.3" y="335.28" size="1.778" layer="95"/>
+</segment>
 </net>
 <net name="N$111" class="0">
@@
 <label x="147.32" y="187.96" size="1.778" layer="95"/>
 </segment>
+<segment>
+<pinref part="CN3" gate="G$1" pin="8"/>
+<wire x1="238.76" y1="320.04" x2="271.78" y2="320.04" width="0.1524" layer="91"/>
+<label x="241.3" y="320.04" size="1.778" layer="95"/>
+</segment>
 </net>
 <net name="ADC_SPI_MISO" class="0">
@@
 <wire x1="144.78" y1="190.5" x2="175.26" y2="190.5" width="0.1524" layer="91"/>
 <label x="147.32" y="190.5" size="1.778" layer="95"/>
+</segment>
+<segment>
+<pinref part="CN3" gate="G$1" pin="6"/>
+<wire x1="238.76" y1="325.12" x2="271.78" y2="325.12" width="0.1524" layer="91"/>
+<label x="241.3" y="325.12" size="1.778" layer="95"/>
 </segment>
 </net>
@@
 </segment>
 </net>
+<net name="DGND" class="0">
+<segment>
+<pinref part="CN3" gate="G$1" pin="10"/>
+<wire x1="238.76" y1="314.96" x2="271.78" y2="314.96" width="0.1524" layer="91"/>
+<label x="241.3" y="314.96" size="1.778" layer="95"/>
+</segment>
+<segment>
+<pinref part="CN3" gate="G$1" pin="11"/>
+<wire x1="238.76" y1="312.42" x2="271.78" y2="312.42" width="0.1524" layer="91"/>
+<label x="241.3" y="312.42" size="1.778" layer="95"/>
+</segment>
+<segment>
+<pinref part="CN3" gate="G$1" pin="12"/>
+<wire x1="238.76" y1="309.88" x2="271.78" y2="309.88" width="0.1524" layer="91"/>
+<label x="241.3" y="309.88" size="1.778" layer="95"/>
+</segment>
+</net>
+<net name="3V3D" class="0">
+<segment>
+<pinref part="CN3" gate="G$1" pin="3"/>
+<wire x1="238.76" y1="332.74" x2="271.78" y2="332.74" width="0.1524" layer="91"/>
+<label x="241.3" y="332.74" size="1.778" layer="95"/>
+</segment>
+<segment>
+<pinref part="CN3" gate="G$1" pin="4"/>
+<wire x1="238.76" y1="330.2" x2="271.78" y2="330.2" width="0.1524" layer="91"/>
+<label x="241.3" y="330.2" size="1.778" layer="95"/>
+</segment>
+</net>
+<net name="ADC_!DRDY" class="0">
+<segment>
+<pinref part="CN3" gate="G$1" pin="7"/>
+<wire x1="238.76" y1="322.58" x2="271.78" y2="322.58" width="0.1524" layer="91"/>
+<label x="241.3" y="322.58" size="1.778" layer="95"/>
+</segment>
+</net>

Commit message: Progress
Parts:
- added TP1, TP2: TEST_POINT_SQUARE, MISC:TEST_POINT_SQUARE
Connections:
- removed net N$83: U1.PA0
- new net N$3: U1.PC4
- new net N$4: TP1.P$1, U6.VIN+
- new net N$5: TP2.P$1, U6.VIN-
- net 3V3: now also U6.VO+
- net DISP_G3: no longer U1.PD3
- net DISP_G7: now also U1.PD3
- net DISP_HSD: no longer U1.PC4
- net DISP_PWM: now also U1.PA0
- net GND: now also U6.COM
Changed lines of the file:
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@@
 <part name="U$43" library="NETS" deviceset="3V3" device=""/>
 <part name="CN3" library="CONNECTORs" deviceset="PICOBLADE_12_" device="TH_V" value="0530471210"/>
+<part name="TP1" library="MISC" deviceset="TEST_POINT_SQUARE" device=""/>
+<part name="TP2" library="MISC" deviceset="TEST_POINT_SQUARE" device=""/>
+<part name="U$15" library="NETS" deviceset="3V3" device=""/>
+<part name="GND15" library="NETS" deviceset="GND" device=""/>
 </parts>
 <sheets>
@@
 <attribute name="VALUE" x="226.06" y="342.9" size="2.286" layer="96"/>
 </instance>
+<instance part="TP1" gate="G$1" x="104.14" y="462.28" smashed="yes" rot="R90">
+<attribute name="NAME" x="101.6" y="462.28" size="1.27" layer="97" rot="R90" align="center"/>
+</instance>
+<instance part="TP2" gate="G$1" x="104.14" y="431.8" smashed="yes" rot="R90">
+<attribute name="NAME" x="101.6" y="431.8" size="1.27" layer="97" rot="R90" align="center"/>
+</instance>
+<instance part="U$15" gate="G$1" x="139.7" y="467.36" smashed="yes">
+<attribute name="VALUE" x="139.7" y="469.9" size="1.778" layer="96" rot="R180" align="center"/>
+</instance>
+<instance part="GND15" gate="G$1" x="139.7" y="441.96" smashed="yes">
+<attribute name="VALUE" x="139.7" y="439.42" size="1.778" layer="96" align="center"/>
+</instance>
 </instances>
 <busses>
@@
 <pinref part="GND54" gate="G$1" pin="GND"/>
 <wire x1="-35.56" y1="25.4" x2="-35.56" y2="22.86" width="0.1524" layer="91"/>
+</segment>
+<segment>
+<pinref part="U6" gate="G$1" pin="COM"/>
+<wire x1="137.16" y1="447.04" x2="139.7" y2="447.04" width="0.1524" layer="91"/>
+<pinref part="GND15" gate="G$1" pin="GND"/>
+<wire x1="139.7" y1="447.04" x2="139.7" y2="444.5" width="0.1524" layer="91"/>
 </segment>
 </net>
@@
 <label x="261.62" y="157.48" size="1.778" layer="95"/>
 </segment>
+<segment>
+<pinref part="U6" gate="G$1" pin="VO+"/>
+<wire x1="137.16" y1="462.28" x2="139.7" y2="462.28" width="0.1524" layer="91"/>
+<pinref part="U$15" gate="G$1" pin="3V3"/>
+<wire x1="139.7" y1="462.28" x2="139.7" y2="464.82" width="0.1524" layer="91"/>
+</segment>
 </net>
 <net name="STM_BOOT0" class="0">
@@
 <label x="76.2" y="147.32" size="1.778" layer="95"/>
 </segment>
+</net>
+<net name="DISP_G4" class="0">
+<segment>
+<pinref part="CN1" gate="G$1" pin="17"/>
+<wire x1="-15.24" y1="182.88" x2="25.4" y2="182.88" width="0.1524" layer="91"/>
+<label x="-12.7" y="182.88" size="1.778" layer="95"/>
+</segment>
+<segment>
+<pinref part="U1" gate="G$1" pin="PB10"/>
+<wire x1="104.14" y1="187.96" x2="73.66" y2="187.96" width="0.1524" layer="91"/>
+<label x="76.2" y="187.96" size="1.778" layer="95"/>
+</segment>
+</net>
+<net name="DISP_G5" class="0">
+<segment>
+<pinref part="CN1" gate="G$1" pin="18"/>
+<wire x1="-15.24" y1="180.34" x2="25.4" y2="180.34" width="0.1524" layer="91"/>
+<label x="-12.7" y="180.34" size="1.778" layer="95"/>
+</segment>
+<segment>
+<pinref part="U1" gate="G$1" pin="PB11"/>
+<wire x1="104.14" y1="185.42" x2="73.66" y2="185.42" width="0.1524" layer="91"/>
+<label x="76.2" y="185.42" size="1.778" layer="95"/>
+</segment>
+</net>
+<net name="DISP_G6" class="0">
+<segment>
+<pinref part="CN1" gate="G$1" pin="19"/>
+<wire x1="-15.24" y1="177.8" x2="25.4" y2="177.8" width="0.1524" layer="91"/>
+<label x="-12.7" y="177.8" size="1.778" layer="95"/>
+</segment>
+<segment>
+<pinref part="U1" gate="G$1" pin="PC7"/>
+<wire x1="104.14" y1="152.4" x2="73.66" y2="152.4" width="0.1524" layer="91"/>
+<label x="76.2" y="152.4" size="1.778" layer="95"/>
+</segment>
+</net>
+<net name="DISP_G7" class="0">
+<segment>
+<pinref part="CN1" gate="G$1" pin="20"/>
+<wire x1="-15.24" y1="175.26" x2="25.4" y2="175.26" width="0.1524" layer="91"/>
+<label x="-12.7" y="175.26" size="1.778" layer="95"/>
+</segment>
 <segment>
 <pinref part="U1" gate="G$1" pin="PD3"/>
@@
 </segment>
 </net>
-<net name="DISP_G4" class="0">
-<segment>
-<pinref part="CN1" gate="G$1" pin="17"/>
-<wire x1="-15.24" y1="182.88" x2="25.4" y2="182.88" width="0.1524" layer="91"/>
-<label x="-12.7" y="182.88" size="1.778" layer="95"/>
-</segment>
-<segment>
-<pinref part="U1" gate="G$1" pin="PB10"/>
-<wire x1="104.14" y1="187.96" x2="73.66" y2="187.96" width="0.1524" layer="91"/>
-<label x="76.2" y="187.96" size="1.778" layer="95"/>
-</segment>
-</net>
-<net name="DISP_G5" class="0">
-<segment>
-<pinref part="CN1" gate="G$1" pin="18"/>
-<wire x1="-15.24" y1="180.34" x2="25.4" y2="180.34" width="0.1524" layer="91"/>
-<label x="-12.7" y="180.34" size="1.778" layer="95"/>
-</segment>
-<segment>
-<pinref part="U1" gate="G$1" pin="PB11"/>
-<wire x1="104.14" y1="185.42" x2="73.66" y2="185.42" width="0.1524" layer="91"/>
-<label x="76.2" y="185.42" size="1.778" layer="95"/>
-</segment>
-</net>
-<net name="DISP_G6" class="0">
-<segment>
-<pinref part="CN1" gate="G$1" pin="19"/>
-<wire x1="-15.24" y1="177.8" x2="25.4" y2="177.8" width="0.1524" layer="91"/>
-<label x="-12.7" y="177.8" size="1.778" layer="95"/>
-</segment>
-<segment>
-<pinref part="U1" gate="G$1" pin="PC7"/>
-<wire x1="104.14" y1="152.4" x2="73.66" y2="152.4" width="0.1524" layer="91"/>
-<label x="76.2" y="152.4" size="1.778" layer="95"/>
-</segment>
-</net>
-<net name="DISP_G7" class="0">
-<segment>
-<pinref part="CN1" gate="G$1" pin="20"/>
-<wire x1="-15.24" y1="175.26" x2="25.4" y2="175.26" width="0.1524" layer="91"/>
-<label x="-12.7" y="175.26" size="1.778" layer="95"/>
-</segment>
-</net>
 <net name="DISP_B0" class="0">
 <segment>
@@
 </segment>
 <segment>
-<pinref part="U1" gate="G$1" pin="PC4"/>
-<wire x1="104.14" y1="160.02" x2="73.66" y2="160.02" width="0.1524" layer="91"/>
-</segment>
-<segment>
 <pinref part="U1" gate="G$1" pin="PC6"/>
 <wire x1="104.14" y1="154.94" x2="73.66" y2="154.94" width="0.1524" layer="91"/>
@@
 <wire x1="144.78" y1="144.78" x2="175.26" y2="144.78" width="0.1524" layer="91"/>
 <label x="147.32" y="144.78" size="1.778" layer="95"/>
-</segment>
-</net>
-<net name="N$83" class="0">
-<segment>
-<pinref part="U1" gate="G$1" pin="PA0"/>
-<wire x1="104.14" y1="256.54" x2="73.66" y2="256.54" width="0.1524" layer="91"/>
 </segment>
 </net>
@@
 <label x="-55.88" y="38.1" size="1.778" layer="95"/>
 </segment>
+<segment>
+<pinref part="U1" gate="G$1" pin="PA0"/>
+<wire x1="104.14" y1="256.54" x2="73.66" y2="256.54" width="0.1524" layer="91"/>
+<label x="76.2" y="256.54" size="1.778" layer="95"/>
+</segment>
 </net>
 <net name="N$86" class="0">
@@
 </segment>
 </net>
+<net name="N$3" class="0">
+<segment>
+<pinref part="U1" gate="G$1" pin="PC4"/>
+<wire x1="104.14" y1="160.02" x2="73.66" y2="160.02" width="0.1524" layer="91"/>
+</segment>
+</net>
+<net name="N$4" class="0">
+<segment>
+<pinref part="U6" gate="G$1" pin="VIN+"/>
+<pinref part="TP1" gate="G$1" pin="P$1"/>
+<wire x1="109.22" y1="462.28" x2="111.76" y2="462.28" width="0.1524" layer="91"/>
+</segment>
+</net>
+<net name="N$5" class="0">
+<segment>
+<pinref part="U6" gate="G$1" pin="VIN-"/>
+<pinref part="TP2" gate="G$1" pin="P$1"/>
+<wire x1="109.22" y1="431.8" x2="111.76" y2="431.8" width="0.1524" layer="91"/>
+</segment>
+</net>
